File: merici-vuz.sch (EAGLE design)
At the start: 0 parts

Commit message: Add first parts of schematics.
Parts:
- added C1, C2: (no value), rcl:C-EUC0805
- added C3: 100nF, rcl:C-EUC0805
- added C4: 10nF, rcl:C-EUC0805
- added C5, C6: 4.7 uF, rcl:CPOL-EUE1.8-4
- added CON-BAT: (no value), pinhead:PINHD-1X2
- added CON-BT: (no value), pinhead:PINHD-1X6
- added CON-OPTO: (no value), pinhead:PINHD-1X3
- added IC1: MEGA328-PB, atmel:MEGA8-AI
- added JP1: (no value), pinhead:PINHD-2X3
- added LED1, LED2, LED3: (no value), led:LEDCHIP-LED0805
- added Q1: 3,6864 MHz, crystal:CRYSTALHC49U70
- added R1, R2, R3: (no value), rcl:R-EU_R0805
- added R4: 10K, rcl:R-EU_R0805
- added R5: 360R, rcl:R-EU_R0805
- added R6: 10k, rcl:R-EU_R0805
- added R7: 680K, rcl:R-EU_R0805
- added R8: 200K, rcl:R-EU_R0805
- added R9: 4K, rcl:R-EU_R0805
- added U$2: MCP73831, mcp73831:MCP73831
- added U1: (no value), microUSB:USB""
Connections:
- new net BAT-SENSE: IC1.PC0(ADC0), R7.1, R8.2
- new net BT-EN: CON-BT.6
- new net BT-RXD: CON-BT.2, IC1.PD1(TXD)
- new net BT-STATE: CON-BT.1
- new net BT-TXD: CON-BT.3, IC1.PD0(RXD)
- new net BT-VCC: CON-BT.5
- new net CHARGE-STAT: U$2.STAT
- new net GND: C1.1, C2.1, C3.2, C4.2, C5.-, C6.-, CON-BAT.2, CON-BT.4, CON-OPTO.2, IC1.GND, IC1.GND@1, IC1.GND@2, JP1.6, R8.1, R9.2, U$2.VSS, U1.GND
- new net LED1: R1.1
- new net LED2: R2.1
- new net LED3: R3.1
- new net MISO: IC1.PB4(MISO), JP1.1
- new net MOSI: IC1.PB3(MOSI/OC2), JP1.4
- new net N$1: C1.2, IC1.PB6(XTAL1/TOSC1), Q1.2
- new net N$10: LED3.C, R3.2
- new net N$2: C2.2, IC1.PB7(XTAL2/TOSC2), Q1.1
- new net N$3: CON-OPTO.3, R5.1
- new net N$4: C4.1, IC1.AREF
- new net N$5: R9.1, U$2.PROG
- new net N$7: C6.+, CON-BAT.1, U$2.VBAT
- new net N$8: LED1.C, R1.2
- new net N$9: LED2.C, R2.2
- new net OPTO-MEASURE: CON-OPTO.1, R4.1
- new net RESET: IC1.PC6(/RESET), JP1.5, R6.2
- new net SCK: IC1.PB5(SCK), JP1.3
- new net VCC: C3.1, IC1.AVCC, IC1.VCC@1, IC1.VCC@2, JP1.2, LED1.A, LED2.A, LED3.A, R4.2, R6.1
- new net VCC-BAT: R7.2
- new net VCC-OPTO: R5.2
- new net VCC-USB: U1.VBUS
- new net VCC/2: C5.+, U$2.VDD

Commit message: Another improvements.
Parts:
- added TP1, TP2, TP3, TP4, TP5, TP6, TP7, TP8, TP9: PTR1B2,54, testpad:PTR1B2,54
- renumbered U$2 to IC2
Connections:
- net BT-EN: now also IC1.PD5(T1)
- net BT-RXD: now also TP7.TP
- net BT-STATE: now also IC1.PD4(XCK/T0)
- net BT-TXD: now also TP8.TP
- net CHARGE-STAT: now also IC1.ADC7
- net GND: now also TP1.TP, TP4.TP, TP6.TP
- net LED1: now also IC1.PC4(ADC4/SDA)
- net LED2: now also IC1.PC5(ADC5/SCL)
- net LED3: now also IC1.ADC6
- net OPTO-MEASURE: now also IC1.PD2(INT0), TP9.TP
- net VCC: now also TP2.TP, TP5.TP
- net VCC/2: now also TP3.TP
Changed lines of the file:
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@@
 <part name="C4" library="rcl" deviceset="C-EU" device="C0805" value="10nF"/>
 <part name="GND8" library="supply1" deviceset="GND" device=""/>
-<part name="U$2" library="mcp73831" deviceset="MCP73831" device=""/>
+<part name="IC2" library="mcp73831" deviceset="MCP73831" device=""/>
 <part name="GND9" library="supply1" deviceset="GND" device=""/>
 <part name="R9" library="rcl" deviceset="R-EU_" device="R0805" value="4K"/>
@@
 <part name="CON-BAT" library="pinhead" deviceset="PINHD-1X2" device=""/>
 <part name="GND11" library="supply1" deviceset="GND" device=""/>
+<part name="TP1" library="testpad" deviceset="PTR1" device="B2,54"/>
+<part name="TP2" library="testpad" deviceset="PTR1" device="B2,54"/>
+<part name="GND12" library="supply1" deviceset="GND" device=""/>
+<part name="P+10" library="supply1" deviceset="VCC" device=""/>
+<part name="TP3" library="testpad" deviceset="PTR1" device="B2,54"/>
+<part name="TP4" library="testpad" deviceset="PTR1" device="B2,54"/>
+<part name="P+11" library="supply1" deviceset="VCC/2" device="" value="VCC-USB"/>
+<part name="GND13" library="supply1" deviceset="GND" device=""/>
+<part name="TP5" library="testpad" deviceset="PTR1" device="B2,54"/>
+<part name="TP6" library="testpad" deviceset="PTR1" device="B2,54"/>
+<part name="SUPPLY2" library="supply2" deviceset="VCC" device="" value="VCC-BAT"/>
+<part name="GND14" library="supply1" deviceset="GND" device=""/>
+<part name="TP7" library="testpad" deviceset="PTR1" device="B2,54"/>
+<part name="TP8" library="testpad" deviceset="PTR1" device="B2,54"/>
+<part name="TP9" library="testpad" deviceset="PTR1" device="B2,54"/>
 </parts>
 <sheets>
@@
 <instance part="C4" gate="G$1" x="33.02" y="147.32"/>
 <instance part="GND8" gate="1" x="33.02" y="104.14"/>
-<instance part="U$2" gate="G$1" x="60.96" y="73.66"/>
+<instance part="IC2" gate="G$1" x="60.96" y="73.66"/>
 <instance part="GND9" gate="1" x="88.9" y="63.5"/>
 <instance part="R9" gate="G$1" x="78.74" y="73.66"/>
@@
 <instance part="CON-BAT" gate="G$1" x="119.38" y="76.2"/>
 <instance part="GND11" gate="1" x="109.22" y="68.58"/>
+<instance part="TP1" gate="G$1" x="231.14" y="60.96" rot="MR180"/>
+<instance part="TP2" gate="G$1" x="231.14" y="76.2"/>
+<instance part="GND12" gate="1" x="231.14" y="53.34"/>
+<instance part="P+10" gate="VCC" x="231.14" y="83.82"/>
+<instance part="TP3" gate="G$1" x="238.76" y="76.2"/>
+<instance part="TP4" gate="G$1" x="238.76" y="60.96" rot="MR180"/>
+<instance part="P+11" gate="G$1" x="238.76" y="83.82"/>
+<instance part="GND13" gate="1" x="238.76" y="53.34"/>
+<instance part="TP5" gate="G$1" x="246.38" y="76.2"/>
+<instance part="TP6" gate="G$1" x="246.38" y="60.96" rot="MR180"/>
+<instance part="SUPPLY2" gate="G$1" x="246.38" y="83.82"/>
+<instance part="GND14" gate="1" x="246.38" y="53.34"/>
+<instance part="TP7" gate="G$1" x="218.44" y="73.66" rot="MR270"/>
+<instance part="TP8" gate="G$1" x="218.44" y="68.58" rot="MR270"/>
+<instance part="TP9" gate="G$1" x="218.44" y="63.5" rot="MR270"/>
 </instances>
 <busses>
@@
 </segment>
 <segment>
-<pinref part="U$2" gate="G$1" pin="VSS"/>
+<pinref part="IC2" gate="G$1" pin="VSS"/>
 <pinref part="GND9" gate="1" pin="GND"/>
 <wire x1="71.12" y1="68.58" x2="88.9" y2="68.58" width="0.1524" layer="91"/>
@@
 <wire x1="109.22" y1="71.12" x2="109.22" y2="76.2" width="0.1524" layer="91"/>
 <pinref part="GND11" gate="1" pin="GND"/>
+</segment>
+<segment>
+<pinref part="TP1" gate="G$1" pin="TP"/>
+<pinref part="GND12" gate="1" pin="GND"/>
+<wire x1="231.14" y1="58.42" x2="231.14" y2="55.88" width="0.1524" layer="91"/>
+</segment>
+<segment>
+<pinref part="TP4" gate="G$1" pin="TP"/>
+<pinref part="GND13" gate="1" pin="GND"/>
+<wire x1="238.76" y1="58.42" x2="238.76" y2="55.88" width="0.1524" layer="91"/>
+</segment>
+<segment>
+<pinref part="TP6" gate="G$1" pin="TP"/>
+<pinref part="GND14" gate="1" pin="GND"/>
+<wire x1="246.38" y1="58.42" x2="246.38" y2="55.88" width="0.1524" layer="91"/>
 </segment>
 </net>
@@
 <pinref part="P+8" gate="VCC" pin="VCC"/>
 </segment>
+<segment>
+<pinref part="TP2" gate="G$1" pin="TP"/>
+<pinref part="P+10" gate="VCC" pin="VCC"/>
+<wire x1="231.14" y1="78.74" x2="231.14" y2="81.28" width="0.1524" layer="91"/>
+</segment>
+<segment>
+<pinref part="TP5" gate="G$1" pin="TP"/>
+<pinref part="SUPPLY2" gate="G$1" pin="VCC"/>
+<wire x1="246.38" y1="78.74" x2="246.38" y2="81.28" width="0.1524" layer="91"/>
+</segment>
 </net>
 <net name="N$8" class="0">
@@
 <label x="228.6" y="129.54" size="1.27" layer="95" rot="R270" xref="yes"/>
 </segment>
+<segment>
+<pinref part="IC1" gate="G$1" pin="PC4(ADC4/SDA)"/>
+<wire x1="91.44" y1="147.32" x2="101.6" y2="147.32" width="0.1524" layer="91"/>
+<label x="101.6" y="147.32" size="1.27" layer="95" xref="yes"/>
+</segment>
 </net>
 <net name="LED2" class="0">
@@
 <label x="236.22" y="129.54" size="1.27" layer="95" rot="R270" xref="yes"/>
 </segment>
+<segment>
+<pinref part="IC1" gate="G$1" pin="PC5(ADC5/SCL)"/>
+<wire x1="91.44" y1="144.78" x2="101.6" y2="144.78" width="0.1524" layer="91"/>
+<label x="101.6" y="144.78" size="1.27" layer="95" xref="yes"/>
+</segment>
 </net>
 <net name="LED3" class="0">
@@
 <wire x1="243.84" y1="134.62" x2="243.84" y2="129.54" width="0.1524" layer="91"/>
 <label x="243.84" y="129.54" size="1.778" layer="95" rot="R270" xref="yes"/>
+</segment>
+<segment>
+<pinref part="IC1" gate="G$1" pin="ADC6"/>
+<wire x1="91.44" y1="142.24" x2="101.6" y2="142.24" width="0.1524" layer="91"/>
+<label x="101.6" y="142.24" size="1.27" layer="95" xref="yes"/>
 </segment>
 </net>
@@
 <label x="71.12" y="33.02" size="1.27" layer="95" xref="yes"/>
 </segment>
+<segment>
+<pinref part="IC1" gate="G$1" pin="PD4(XCK/T0)"/>
+<wire x1="91.44" y1="124.46" x2="101.6" y2="124.46" width="0.1524" layer="91"/>
+<label x="101.6" y="124.46" size="1.27" layer="95" xref="yes"/>
+</segment>
 </net>
 <net name="BT-RXD" class="0">
@@
 <label x="101.6" y="132.08" size="1.27" layer="95" xref="yes"/>
 </segment>
+<segment>
+<pinref part="TP7" gate="G$1" pin="TP"/>
+<wire x1="215.9" y1="73.66" x2="213.36" y2="73.66" width="0.1524" layer="91"/>
+<label x="213.36" y="73.66" size="1.27" layer="95" rot="MR0" xref="yes"/>
+</segment>
 </net>
 <net name="BT-TXD" class="0">
@@
 <label x="101.6" y="134.62" size="1.27" layer="95" xref="yes"/>
 </segment>
+<segment>
+<pinref part="TP8" gate="G$1" pin="TP"/>
+<wire x1="215.9" y1="68.58" x2="213.36" y2="68.58" width="0.1524" layer="91"/>
+<label x="213.36" y="68.58" size="1.27" layer="95" rot="R180" xref="yes"/>
+</segment>
 </net>
 <net name="BT-EN" class="0">
@@
 <wire x1="55.88" y1="20.32" x2="71.12" y2="20.32" width="0.1524" layer="91"/>
 <label x="71.12" y="20.32" size="1.27" layer="95" xref="yes"/>
+</segment>
+<segment>
+<pinref part="IC1" gate="G$1" pin="PD5(T1)"/>
+<wire x1="91.44" y1="121.92" x2="101.6" y2="121.92" width="0.1524" layer="91"/>
+<label x="101.6" y="121.92" size="1.27" layer="95" xref="yes"/>
 </segment>
 </net>
@@
 <label x="129.54" y="27.94" size="1.27" layer="95" xref="yes"/>
 </segment>
+<segment>
+<pinref part="TP9" gate="G$1" pin="TP"/>
+<wire x1="215.9" y1="63.5" x2="213.36" y2="63.5" width="0.1524" layer="91"/>
+<label x="213.36" y="63.5" size="1.27" layer="95" rot="R180" xref="yes"/>
+</segment>
+<segment>
+<pinref part="IC1" gate="G$1" pin="PD2(INT0)"/>
+<wire x1="91.44" y1="129.54" x2="101.6" y2="129.54" width="0.1524" layer="91"/>
+<label x="101.6" y="129.54" size="1.27" layer="95" xref="yes"/>
+</segment>
 </net>
 <net name="MISO" class="0">
@@
 <segment>
 <pinref part="R9" gate="G$1" pin="1"/>
-<pinref part="U$2" gate="G$1" pin="PROG"/>
+<pinref part="IC2" gate="G$1" pin="PROG"/>
 <wire x1="73.66" y1="73.66" x2="71.12" y2="73.66" width="0.1524" layer="91"/>
 </segment>
@@
 <net name="CHARGE-STAT" class="0">
 <segment>
-<pinref part="U$2" gate="G$1" pin="STAT"/>
+<pinref part="IC2" gate="G$1" pin="STAT"/>
 <wire x1="50.8" y1="71.12" x2="48.26" y2="71.12" width="0.1524" layer="91"/>
 <label x="48.26" y="71.12" size="1.27" layer="95" rot="R180" xref="yes"/>
 </segment>
+<segment>
+<pinref part="IC1" gate="G$1" pin="ADC7"/>
+<wire x1="91.44" y1="139.7" x2="101.6" y2="139.7" width="0.1524" layer="91"/>
+<label x="101.6" y="139.7" size="1.27" layer="95" xref="yes"/>
+</segment>
 </net>
 <net name="VCC/2" class="0">
 <segment>
-<pinref part="U$2" gate="G$1" pin="VDD"/>
+<pinref part="IC2" gate="G$1" pin="VDD"/>
 <wire x1="50.8" y1="76.2" x2="27.94" y2="76.2" width="0.1524" layer="91"/>
 <pinref part="P+9" gate="G$1" pin="VCC/2"/>
@@
 <junction x="27.94" y="76.2"/>
 </segment>
+<segment>
+<pinref part="TP3" gate="G$1" pin="TP"/>
+<pinref part="P+11" gate="G$1" pin="VCC/2"/>
+<wire x1="238.76" y1="78.74" x2="238.76" y2="81.28" width="0.1524" layer="91"/>
+</segment>
 </net>
 <net name="N$7" class="0">
 <segment>
-<pinref part="U$2" gate="G$1" pin="VBAT"/>
+<pinref part="IC2" gate="G$1" pin="VBAT"/>
 <pinref part="C6" gate="A" pin="+"/>
 <wire x1="71.12" y1="78.74" x2="93.98" y2="78.74" width="0.1524" layer="91"/>
