File: merici-vuz.sch (EAGLE design)
At the start: 53 parts, among them IC1 MEGA328-PB, IC2 MCP73831, IC3 LE33, Q1 3,6864 MHz, Q4 TSM2302CX, T1 IRF7306

Commit message: Remove unwanted VCC/2.
Connections:
- removed net VCC/2: C5.1, IC2.VDD, LED4.A, TP3.TP
- net VCC-USB: now also C5.1, IC2.VDD, LED4.A, TP3.TP

Commit message: First prototype of PCB.
Parts:
- Q1: device crystal:CRYSTALHC49U70 -> crystal:CRYSTALHC49UP
- S-OFF, S-ON: value (none) -> P-DT2112C; device switch-omron:10-XX -> switch-tact:DTSM-3
- TP1, TP2, TP3, TP4, TP5, TP6, TP7, TP8, TP9: value PTR1B2,54 -> PTR1B1,27; device testpad:PTR1B2,54 -> testpad:PTR1B1,27
Connections:
- removed net RESET: CON-PROG.5
- net !RESET: now also CON-PROG.5
- net !SHUTDOWN: now also IC1.PB2(SS/OC1B); no longer IC1.PC1(ADC1)
- net !SHUTDOWN_INT: now also S-OFF.1; no longer S-OFF.S, S-OFF.S1
- net BT-EN: now also IC1.PC4(ADC4/SDA); no longer IC1.PD5(T1)
- net CR1: now also IC1.PB7(XTAL2/TOSC2); no longer IC1.PB6(XTAL1/TOSC1)
- net CR2: now also IC1.PB6(XTAL1/TOSC1); no longer IC1.PB7(XTAL2/TOSC2)
- net GND: now also S-OFF.2, S-ON.1; no longer S-OFF.P, S-OFF.P1, S-ON.P, S-ON.P1
- net LED-GR: now also IC1.PC1(ADC1); no longer IC1.ADC6
- net LED-RED: now also IC1.PC3(ADC3); no longer IC1.PC4(ADC4/SDA)
- net LED-YEL: now also IC1.PC2(ADC2); no longer IC1.PC5(ADC5/SCL)
- net START_BUTTON: now also S-ON.2; no longer S-ON.S, S-ON.S1
- net VCC: no longer TP5.TP
- net VCC-BAT: now also TP5.TP
Other:
- moved on the sheet: C1, C2, Q1
